File: KiCAD/supercharger/supercharger.kicad_sch (KiCad schematic)
At the start: 25 parts, among them J2 BAT, J4 UJC-H-G-SMT-1-P6-TR, U1 STC4054, U2 HM1160

Commit message: Round-off tracks
Parts:
- D2: footprint SOT95P280X145-5N -> Package_TO_SOT_SMD:SOT-23-5_HandSoldering
- D3: footprint SOT95P248X115-3N -> Package_TO_SOT_SMD:SOT-23-3
Changed lines of the file:
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@@
 			)
 		)
-		(property "Footprint" "SOT95P280X145-5N"
+		(property "Footprint" "Package_TO_SOT_SMD:SOT-23-5_HandSoldering"
 			(at 168.91 126.67 0)
 			(effects
@@
 			)
 		)
-		(property "Footprint" "SOT95P248X115-3N"
+		(property "Footprint" "Package_TO_SOT_SMD:SOT-23-3"
 			(at 289.23 60.96 0)
 			(effects
